File: Backplane - Balance.kicad_pcb (KiCad board)
At the start: 2 copper layers, 100 x 280.5 mm, 61 parts, among them J1 IDC Balence Connector, J2 IDC Balence Connector, U1 DS18B20, U2 DS18B20

Commit message: Last changes for V1
Routing:
- net /CELL9: track 86.4 -> 77.7 mm
