File: Backplane.kicad_pcb (KiCad board)
At the start: 2 copper layers, 100 x 280.5 mm, 12 parts, among them J1 IDC Balence Connector, J2 IDC Balence Connector, U1 DS18B20, U2 DS18B20

Commit message: Reroute using TopoR
Routing:
- net /CELL12: track 99.8 -> 217.3 mm, vias 4 -> 1
- net /CELL10: track 61.4 -> 149.2 mm, vias 4 -> 0
- net /CELL8: track 78.4 -> 164.6 mm, vias 4 -> 1
- net /CELL6: track 57.5 -> 126.6 mm, vias 2 -> 0
- net /CELL4: track 70.9 -> 138.4 mm, vias 5 -> 1
- net /CELL2: track 103.1 -> 166.4 mm, vias 5 -> 0
- net GND: track 341.5 -> 300.3 mm, vias 3 -> 2
- net /CELL3: track 154.7 -> 117.0 mm, vias 3 -> 1
- net VBUS: track 199.0 -> 162.9 mm, vias 0 -> 1
- net /CELL13: track 177.6 -> 151.0 mm, vias 2 -> 1
- net /CELL7: track 82.4 -> 55.9 mm, vias 1 -> 0
- net /CELL11: track 140.8 -> 164.7 mm, vias 2 -> 0
- net /CELL1: track 178.3 -> 154.7 mm, vias 1 -> 0
- net /CELL5: track 114.8 -> 91.5 mm
- net /CELL9: track 108.1 -> 87.0 mm, vias 3 -> 0
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- added copper zone on B.Cu, net (none)
- added copper zone on F.Cu, net (none)
- removed copper zone on B.Cu, net GND
- removed copper zone on F.Cu, net GND

Commit message: - Added Balance Version - Added Images - Added Battery .step
Parts:
- added kibuzzard-680EEA00: G***, kibuzzard-680EEA00, F.Cu at (66.0, 33.0)
- added kibuzzard-680EEA00: G***, kibuzzard-680EEA00, F.Cu at (49.0, 234.0)
- added kibuzzard-680EEA19: G***, kibuzzard-680EEA19, F.Cu at (69.0, 33.3)
- added kibuzzard-680EEA19: G***, kibuzzard-680EEA19, F.Cu at (46.0, 234.0)
- added kibuzzard-680EEA42: G***, kibuzzard-680EEA42, F.Cu at (52.0, 234.0)
- added kibuzzard-680EEA42: G***, kibuzzard-680EEA42, F.Cu at (63.0, 32.8)
- added kibuzzard-680EEAED: G***, kibuzzard-680EEAED, F.Cu at (74.0, 260.0)
- added kibuzzard-680EF0B4: G***, kibuzzard-680EF0B4, F.Cu at (50.0, 250.0)
- added kibuzzard-680EF17D: G***, kibuzzard-680EF17D, F.Cu at (50.0, 210.0)
- added kibuzzard-680EF18E: G***, kibuzzard-680EF18E, F.Cu at (50.0, 170.0)
- added kibuzzard-680EF1BA: G***, kibuzzard-680EF1BA, F.Cu at (50.0, 120.0)
- added kibuzzard-680EF1E5: G***, kibuzzard-680EF1E5, F.Cu at (50.0, 90.0)
- added kibuzzard-680EF203: G***, kibuzzard-680EF203, F.Cu at (50.0, 50.0)
- added kibuzzard-680EF230: G***, kibuzzard-680EF230, F.Cu at (50.0, 10.0)
- added kibuzzard-680EF2D1: G***, kibuzzard-680EF2D1, F.Cu at (29.0, 240.0)
- added kibuzzard-680EF2FD: G***, kibuzzard-680EF2FD, F.Cu at (30.0, 160.0)
- added kibuzzard-680EF343: G***, kibuzzard-680EF343, F.Cu at (30.0, 80.0)
- added kibuzzard-680EF361: G***, kibuzzard-680EF361, F.Cu at (31.0, 20.0)
- added kibuzzard-680EF474: G***, kibuzzard-680EF474, F.Cu at (70.0, 200.0)
- added kibuzzard-680EF51A: G***, kibuzzard-680EF51A, F.Cu at (70.0, 120.0)
- added kibuzzard-680EF59B: G***, kibuzzard-680EF59B, F.Cu at (69.0, 44.0)
